Commit message: CAMERA FIXED

File: src/snake_bot/urdf/camera.xacro (robot description, xacro)
@@ -2,7 +2,7 @@
 <robot xmlns:xacro="http://www.ros.org/wiki/xacro" >
     <joint name="camera_joint" type="fixed">
-        <parent link="link_1"/>
+        <parent link="link_10"/>
         <child link="camera_link"/>
-        <origin xyz="0 0 0.03" rpy="0 0 ${-pi/2}"/>
+        <origin xyz="0 0.14 0.03" rpy="0 ${-pi/18} ${pi/2}"/>
     </joint>
     <link name="camera_link">

File: src/snake_bot/urdf/ros2_control.xacro (robot description, xacro)
@@ -29,5 +29,5 @@
     </gazebo>
     <gazebo reference="link_10">
-        <material>Gazebo/Orange</material>
+        <material>Gazebo/Pink</material>
     </gazebo>
     <ros2_control name="GazeboSystem" type="system">
