Commit message: new URDF for 3 obstacle paper

File: src/snake_bot/urdf/snakebot.xacro (robot description, xacro)
@@ -66,5 +66,5 @@
         <child link="link_3"/>
         <limit lower="-0.785398163397" upper="0.785398163397" velocity="50.0" effort="1000.0"/>
-        <origin xyz="0.0 0.175 0.0" rpy="0 0 0"/>
+        <origin xyz="0.0 0.175 0.0" rpy="0 0 -45"/>
         <axis xyz="0 0 1"/>
         <joint_properties damping="6.0" friction="6.0"/>
@@ -148,5 +148,5 @@
         <child link="link_6"/>
         <limit lower="-0.785398163397" upper="0.785398163397" velocity="50.0" effort="1000.0"/>
-        <origin xyz="0.0 0.175 0.0" rpy="0 0 0"/>
+        <origin xyz="0.0 0.175 0.0" rpy="0 0 -20"/>
         <axis xyz="0 0 1"/>
         <joint_properties damping="6.0" friction="6.0"/>
@@ -260,5 +260,5 @@
         <child link="link_10"/>
         <limit lower="-0.785398163397" upper="0.785398163397" velocity="50.0" effort="1000.0"/>
-        <origin xyz="0.0 0.175 0.0" rpy="0 0 0"/>
+        <origin xyz="0.0 0.175 0.0" rpy="0 0 -20"/>
         <axis xyz="0 0 1"/>
         <joint_properties damping="6.0" friction="6.0"/>

Commit message: immovable obstacles and right angles

File: src/snake_bot/urdf/snakebot.xacro (robot description, xacro)
@@ -66,5 +66,5 @@
         <child link="link_3"/>
         <limit lower="-0.785398163397" upper="0.785398163397" velocity="50.0" effort="1000.0"/>
-        <origin xyz="0.0 0.175 0.0" rpy="0 0 -45"/>
+        <origin xyz="0.0 0.175 0.0" rpy="0 0 -1.0472"/>
         <axis xyz="0 0 1"/>
         <joint_properties damping="6.0" friction="6.0"/>
@@ -148,5 +148,5 @@
         <child link="link_6"/>
         <limit lower="-0.785398163397" upper="0.785398163397" velocity="50.0" effort="1000.0"/>
-        <origin xyz="0.0 0.175 0.0" rpy="0 0 -20"/>
+        <origin xyz="0.0 0.175 0.0" rpy="0 0 -1.0472"/>
         <axis xyz="0 0 1"/>
         <joint_properties damping="6.0" friction="6.0"/>
@@ -232,5 +232,5 @@
         <child link="link_9"/>
         <limit lower="-0.785398163397" upper="0.785398163397" velocity="50.0" effort="1000.0"/>
-        <origin xyz="0.0 0.175 0.0" rpy="0 0 0"/>
+        <origin xyz="0.0 0.175 0.0" rpy="0 0 0.174533"/>
         <axis xyz="0 0 1"/>
         <joint_properties damping="6.0" friction="6.0"/>
@@ -260,5 +260,5 @@
         <child link="link_10"/>
         <limit lower="-0.785398163397" upper="0.785398163397" velocity="50.0" effort="1000.0"/>
-        <origin xyz="0.0 0.175 0.0" rpy="0 0 -20"/>
+        <origin xyz="0.0 0.175 0.0" rpy="0 0 0.174533"/>
         <axis xyz="0 0 1"/>
         <joint_properties damping="6.0" friction="6.0"/>

Commit message: 2 obstacles world introduced

File: src/snake_bot/urdf/snakebot.xacro (robot description, xacro)
@@ -38,5 +38,5 @@
         <child link="link_2"/>
         <limit lower="-0.785398163397" upper="0.785398163397" velocity="50.0" effort="1000.0"/>
-        <origin xyz="0.0 0.175 0.0" rpy="0 0 0"/>
+        <origin xyz="0.0 0.175 0.0" rpy="0 0 -0.349066"/>
         <axis xyz="0 0 1"/>
         <joint_properties damping="6.0" friction="6.0"/>
@@ -66,5 +66,5 @@
         <child link="link_3"/>
         <limit lower="-0.785398163397" upper="0.785398163397" velocity="50.0" effort="1000.0"/>
-        <origin xyz="0.0 0.175 0.0" rpy="0 0 -1.0472"/>
+        <origin xyz="0.0 0.175 0.0" rpy="0 0 -0.349066"/>
         <axis xyz="0 0 1"/>
         <joint_properties damping="6.0" friction="6.0"/>
@@ -94,5 +94,5 @@
         <child link="link_4"/>
         <limit lower="-0.785398163397" upper="0.785398163397" velocity="50.0" effort="1000.0"/>
-        <origin xyz="0.0 0.175 0.0" rpy="0 0 0"/>
+        <origin xyz="0.0 0.175 0.0" rpy="0 0 -0.349066"/>
         <axis xyz="0 0 1"/>
         <joint_properties damping="6.0" friction="6.0"/>
@@ -121,5 +121,5 @@
         <child link="link_5"/>
         <limit lower="-0.785398163397" upper="0.785398163397" velocity="50.0" effort="1000.0"/>
-        <origin xyz="0.0 0.175 0.0" rpy="0 0 0"/>
+        <origin xyz="0.0 0.175 0.0" rpy="0 0 -0.349066"/>
         <axis xyz="0 0 1"/>
         <joint_properties damping="6.0" friction="6.0"/>
@@ -148,5 +148,5 @@
         <child link="link_6"/>
         <limit lower="-0.785398163397" upper="0.785398163397" velocity="50.0" effort="1000.0"/>
-        <origin xyz="0.0 0.175 0.0" rpy="0 0 -1.0472"/>
+        <origin xyz="0.0 0.175 0.0" rpy="0 0 -0.349066"/>
         <axis xyz="0 0 1"/>
         <joint_properties damping="6.0" friction="6.0"/>
@@ -176,5 +176,5 @@
         <child link="link_7"/>
         <limit lower="-0.785398163397" upper="0.785398163397" velocity="50.0" effort="1000.0"/>
-        <origin xyz="0.0 0.175 0.0" rpy="0 0 0"/>
+        <origin xyz="0.0 0.175 0.0" rpy="0 0 -0.349066"/>
         <axis xyz="0 0 1"/>
         <joint_properties damping="6.0" friction="6.0"/>
@@ -204,5 +204,5 @@
         <child link="link_8"/>
         <limit lower="-0.785398163397" upper="0.785398163397" velocity="50.0" effort="1000.0"/>
-        <origin xyz="0.0 0.175 0.0" rpy="0 0 0"/>
+        <origin xyz="0.0 0.175 0.0" rpy="0 0 -0.349066"/>
         <axis xyz="0 0 1"/>
         <joint_properties damping="6.0" friction="6.0"/>
@@ -232,5 +232,5 @@
         <child link="link_9"/>
         <limit lower="-0.785398163397" upper="0.785398163397" velocity="50.0" effort="1000.0"/>
-        <origin xyz="0.0 0.175 0.0" rpy="0 0 0.174533"/>
+        <origin xyz="0.0 0.175 0.0" rpy="0 0 -0.349066"/>
         <axis xyz="0 0 1"/>
         <joint_properties damping="6.0" friction="6.0"/>
@@ -260,5 +260,5 @@
         <child link="link_10"/>
         <limit lower="-0.785398163397" upper="0.785398163397" velocity="50.0" effort="1000.0"/>
-        <origin xyz="0.0 0.175 0.0" rpy="0 0 0.174533"/>
+        <origin xyz="0.0 0.175 0.0" rpy="0 0 -0.349066"/>
         <axis xyz="0 0 1"/>
         <joint_properties damping="6.0" friction="6.0"/>

Commit message: Obstacles aligned and extra files deleted

File: src/snake_bot/urdf/snakebot.xacro (robot description, xacro)
@@ -66,5 +66,5 @@
         <child link="link_3"/>
         <limit lower="-0.785398163397" upper="0.785398163397" velocity="50.0" effort="1000.0"/>
-        <origin xyz="0.0 0.175 0.0" rpy="0 0 -1.0472"/>
+        <origin xyz="0.0 0.175 0.0" rpy="0 0 -1.309"/>
         <axis xyz="0 0 1"/>
         <joint_properties damping="6.0" friction="6.0"/>
@@ -148,5 +148,5 @@
         <child link="link_6"/>
         <limit lower="-0.785398163397" upper="0.785398163397" velocity="50.0" effort="1000.0"/>
-        <origin xyz="0.0 0.175 0.0" rpy="0 0 -1.0472"/>
+        <origin xyz="0.0 0.175 0.0" rpy="0 0 -1.22173"/>
         <axis xyz="0 0 1"/>
         <joint_properties damping="6.0" friction="6.0"/>
@@ -176,5 +176,5 @@
         <child link="link_7"/>
         <limit lower="-0.785398163397" upper="0.785398163397" velocity="50.0" effort="1000.0"/>
-        <origin xyz="0.0 0.175 0.0" rpy="0 0 0"/>
+        <origin xyz="0.0 0.175 0.0" rpy="0 0 -0.174533"/>
         <axis xyz="0 0 1"/>
         <joint_properties damping="6.0" friction="6.0"/>
@@ -204,5 +204,5 @@
         <child link="link_8"/>
         <limit lower="-0.785398163397" upper="0.785398163397" velocity="50.0" effort="1000.0"/>
-        <origin xyz="0.0 0.175 0.0" rpy="0 0 0"/>
+        <origin xyz="0.0 0.175 0.0" rpy="0 0 -0.174533"/>
         <axis xyz="0 0 1"/>
         <joint_properties damping="6.0" friction="6.0"/>
@@ -232,5 +232,5 @@
         <child link="link_9"/>
         <limit lower="-0.785398163397" upper="0.785398163397" velocity="50.0" effort="1000.0"/>
-        <origin xyz="0.0 0.175 0.0" rpy="0 0 0.174533"/>
+        <origin xyz="0.0 0.175 0.0" rpy="0 0 -0.174533"/>
         <axis xyz="0 0 1"/>
         <joint_properties damping="6.0" friction="6.0"/>
@@ -260,5 +260,5 @@
         <child link="link_10"/>
         <limit lower="-0.785398163397" upper="0.785398163397" velocity="50.0" effort="1000.0"/>
-        <origin xyz="0.0 0.175 0.0" rpy="0 0 0.174533"/>
+        <origin xyz="0.0 0.175 0.0" rpy="0 0 -1.309"/>
         <axis xyz="0 0 1"/>
         <joint_properties damping="6.0" friction="6.0"/>

Commit message: sensors worknig and configured for all elementst

File: src/snake_bot/urdf/snakebot.xacro (robot description, xacro)
@@ -23,5 +23,5 @@
             <material name="green"/>
         </visual>
-        <collision>
+        <collision name="link_1_collision">
             <origin xyz="0.0 0.07 0.03" rpy="0.0 0.0 0"/>
             <geometry>
@@ -51,5 +51,5 @@
             </geometry>
         </visual>
-        <collision>
+        <collision name="link_2_collision">
             <origin xyz="0.0 0.07 0.03" rpy="0.0 0.0 0.0"/>
             <geometry>
@@ -79,5 +79,5 @@
             </geometry>
         </visual>
-        <collision>
+        <collision name="link_3_collision">
             <origin xyz="0.0 0.07 0.03" rpy="0.0 0.0 0.0"/>
             <geometry>
@@ -107,5 +107,5 @@
             </geometry>
         </visual>
-        <collision>
+        <collision name="link_4_collision">
             <origin xyz="0.0 0.07 0.03" rpy="0.0 0.0 0.0"/>
             <geometry>
@@ -134,5 +134,5 @@
             </geometry>
         </visual>
-        <collision>
+        <collision name="link_5_collision">
             <origin xyz="0.0 0.07 0.03" rpy="0.0 0.0 0.0"/>
             <geometry>
@@ -161,5 +161,5 @@
             </geometry>
         </visual>
-        <collision>
+        <collision name="link_6_collision">
             <origin xyz="0.0 0.07 0.03" rpy="0.0 0.0 0.0"/>
             <geometry>
@@ -189,5 +189,5 @@
             </geometry>
         </visual>
-        <collision>
+        <collision name="link_7_collision">
             <origin xyz="0.0 0.07 0.03" rpy="0.0 0.0 0.0"/>
             <geometry>
@@ -217,5 +217,5 @@
             </geometry>
         </visual>
-        <collision>
+        <collision name="link_8_collision">
             <origin xyz="0.0 0.07 0.03" rpy="0.0 0.0 0.0"/>
             <geometry>
@@ -245,5 +245,5 @@
             </geometry>
         </visual>
-        <collision>
+        <collision name="link_9_collision">
             <origin xyz="0.0 0.07 0.03" rpy="0.0 0.0 0.0"/>
             <geometry>
@@ -273,5 +273,5 @@
             </geometry>
         </visual>
-        <collision>
+        <collision name="link_10_collision">
             <origin xyz="0.0 0.07 0.03" rpy="0.0 0.0 0.0"/>
             <geometry>

Commit message: obstacles updated and added

File: src/snake_bot/urdf/snakebot.xacro (robot description, xacro)
@@ -12,5 +12,5 @@
       <parent link="base_link"/>
       <child link="link_1"/>
-      <origin xyz="0.0 0 0.0" rpy="0 0 0.523599"/>
+      <origin xyz="0.0 0 0.0" rpy="0 0 0.436332"/>
     </joint>
     <!--LINK_1 -->
@@ -176,5 +176,5 @@
         <child link="link_7"/>
         <limit lower="-0.785398163397" upper="0.785398163397" velocity="50.0" effort="1000.0"/>
-        <origin xyz="0.0 0.175 0.0" rpy="0 0 -0.174533"/>
+        <origin xyz="0.0 0.175 0.0" rpy="0 0 0"/>
         <axis xyz="0 0 1"/>
         <joint_properties damping="6.0" friction="6.0"/>
@@ -283,18 +283,3 @@
         </xacro:inertial_box>
     </link>
-    <!--gazebo>
-          <plugin name="gazebo_ros_joint_state_publisher"
-                    filename="libgazebo_ros_joint_state_publisher.so">
-                    <update_rate>50</update_rate>
-                    <joint_name>link_1_2_joint</joint_name>
-                    <joint_name>link_2_3_joint</joint_name>
-                    <joint_name>link_3_4_joint</joint_name>
-                    <joint_name>link_4_5_joint</joint_name>
-                    <joint_name>link_5_6_joint</joint_name>
-                    <joint_name>link_6_7_joint</joint_name>
-                    <joint_name>link_7_8_joint</joint_name>
-                    <joint_name>link_8_9_joint</joint_name>
-                    <joint_name>link_9_10_joint</joint_name>
-        </plugin>
-    </gazebo-->
 </robot>

Commit message: obstacles updated and added

File: src/snake_bot/urdf/snakebot.xacro (robot description, xacro)
@@ -12,5 +12,5 @@
       <parent link="base_link"/>
       <child link="link_1"/>
-      <origin xyz="0.0 0 0.0" rpy="0 0 0"/>
+      <origin xyz="0.0 0 0.0" rpy="0 0 0.523599"/>
      </joint>
     <!--LINK_1 -->
@@ -38,5 +38,5 @@
         <child link="link_2"/>
         <limit lower="-0.785398163397" upper="0.785398163397" velocity="50.0" effort="1000.0"/>
-        <origin xyz="0.0 0.175 0.0" rpy="0 0 -0.349066"/>
+        <origin xyz="0.0 0.175 0.0" rpy="0 0 -0.4363326"/>
         <axis xyz="0 0 1"/>
         <joint_properties damping="6.0" friction="6.0"/>
@@ -66,5 +66,5 @@
         <child link="link_3"/>
         <limit lower="-0.785398163397" upper="0.785398163397" velocity="50.0" effort="1000.0"/>
-        <origin xyz="0.0 0.175 0.0" rpy="0 0 -0.349066"/>
+        <origin xyz="0.0 0.175 0.0" rpy="0 0 -0.4363326"/>
         <axis xyz="0 0 1"/>
         <joint_properties damping="6.0" friction="6.0"/>
@@ -94,5 +94,5 @@
         <child link="link_4"/>
         <limit lower="-0.785398163397" upper="0.785398163397" velocity="50.0" effort="1000.0"/>
-        <origin xyz="0.0 0.175 0.0" rpy="0 0 -0.349066"/>
+        <origin xyz="0.0 0.175 0.0" rpy="0 0 -0.4363326"/>
         <axis xyz="0 0 1"/>
         <joint_properties damping="6.0" friction="6.0"/>
@@ -121,5 +121,5 @@
         <child link="link_5"/>
         <limit lower="-0.785398163397" upper="0.785398163397" velocity="50.0" effort="1000.0"/>
-        <origin xyz="0.0 0.175 0.0" rpy="0 0 -0.349066"/>
+        <origin xyz="0.0 0.175 0.0" rpy="0 0 -0.4363326"/>
         <axis xyz="0 0 1"/>
         <joint_properties damping="6.0" friction="6.0"/>
@@ -148,5 +148,5 @@
         <child link="link_6"/>
         <limit lower="-0.785398163397" upper="0.785398163397" velocity="50.0" effort="1000.0"/>
-        <origin xyz="0.0 0.175 0.0" rpy="0 0 -0.349066"/>
+        <origin xyz="0.0 0.175 0.0" rpy="0 0 -0.4363326"/>
         <axis xyz="0 0 1"/>
         <joint_properties damping="6.0" friction="6.0"/>
@@ -176,5 +176,5 @@
         <child link="link_7"/>
         <limit lower="-0.785398163397" upper="0.785398163397" velocity="50.0" effort="1000.0"/>
-        <origin xyz="0.0 0.175 0.0" rpy="0 0 -0.349066"/>
+        <origin xyz="0.0 0.175 0.0" rpy="0 0 -0.4363326"/>
         <axis xyz="0 0 1"/>
         <joint_properties damping="6.0" friction="6.0"/>
@@ -204,5 +204,5 @@
         <child link="link_8"/>
         <limit lower="-0.785398163397" upper="0.785398163397" velocity="50.0" effort="1000.0"/>
-        <origin xyz="0.0 0.175 0.0" rpy="0 0 -0.349066"/>
+        <origin xyz="0.0 0.175 0.0" rpy="0 0 -0.4363326"/>
         <axis xyz="0 0 1"/>
         <joint_properties damping="6.0" friction="6.0"/>
@@ -232,5 +232,5 @@
         <child link="link_9"/>
         <limit lower="-0.785398163397" upper="0.785398163397" velocity="50.0" effort="1000.0"/>
-        <origin xyz="0.0 0.175 0.0" rpy="0 0 -0.349066"/>
+        <origin xyz="0.0 0.175 0.0" rpy="0 0 -0.4363326"/>
         <axis xyz="0 0 1"/>
         <joint_properties damping="6.0" friction="6.0"/>
@@ -260,5 +260,5 @@
         <child link="link_10"/>
         <limit lower="-0.785398163397" upper="0.785398163397" velocity="50.0" effort="1000.0"/>
-        <origin xyz="0.0 0.175 0.0" rpy="0 0 -0.349066"/>
+        <origin xyz="0.0 0.175 0.0" rpy="0 0 -0.4363326"/>
         <axis xyz="0 0 1"/>
         <joint_properties damping="6.0" friction="6.0"/>
@@ -283,18 +283,3 @@
         </xacro:inertial_box>
     </link>
-    <!--gazebo>
-          <plugin name="gazebo_ros_joint_state_publisher"
-                    filename="libgazebo_ros_joint_state_publisher.so">
-                    <update_rate>50</update_rate>
-                    <joint_name>link_1_2_joint</joint_name>
-                    <joint_name>link_2_3_joint</joint_name>
-                    <joint_name>link_3_4_joint</joint_name>
-                    <joint_name>link_4_5_joint</joint_name>
-                    <joint_name>link_5_6_joint</joint_name>
-                    <joint_name>link_6_7_joint</joint_name>
-                    <joint_name>link_7_8_joint</joint_name>
-                    <joint_name>link_8_9_joint</joint_name>
-                    <joint_name>link_9_10_joint</joint_name>
-        </plugin>
-    </gazebo-->
 </robot>
