Commit message: commit

File: src/snake_bot/urdf/ros2_control.xacro (robot description, xacro)
@@ -1,5 +1,5 @@
 <?xml version="1.0"?>
 <robot xmlns:xacro="http://www.ros.org/wiki/xacro"  >
-     <gazebo reference="link_1">
+    <gazebo reference="link_1">
         <material>Gazebo/Green</material>
     </gazebo>
@@ -31,85 +31,85 @@
         <material>Gazebo/Orange</material>
     </gazebo>
-  <ros2_control name="GazeboSystem" type="system">
+    <ros2_control name="GazeboSystem" type="system">
     	<hardware>
             <plugin>gazebo_ros2_control/GazeboSystem</plugin>
     	</hardware>
 <!--  ****************************************************** * * * BELOW IS Commented * *************************************************************************************** * * * * * -->
-    <joint name="link_1_2_joint">
-        <command_interface name="effort">
-            <param name="min">0</param>
-            <param name="max">200</param>
-        </command_interface>
-        <state_interface name="position"/>
-    </joint>
-    <joint name="link_2_3_joint">
-        <command_interface name="effort">
-            <param name="min">0</param>
-            <param name="max">200</param>
-        </command_interface>
-        <state_interface name="position"/>
-    </joint>
-    <joint name="link_3_4_joint">
-        <command_interface name="effort">
-            <param name="min">0</param>
-            <param name="max">200</param>
-        </command_interface>
-        <state_interface name="position"/>
-    </joint>
-    <joint name="link_4_5_joint">
-        <command_interface name="effort">
-            <param name="min">0</param>
-            <param name="max">200</param>
-        </command_interface>
-        <state_interface name="position"/>
-    </joint>
-    <joint name="link_5_6_joint">
-        <command_interface name="effort">
-            <param name="min">0</param>
-            <param name="max">200</param>
-        </command_interface>
-        <state_interface name="position"/>
-    </joint>
-    <joint name="link_6_7_joint">
-        <command_interface name="effort">
-            <param name="min">0</param>
-            <param name="max">200</param>
-        </command_interface>
-        <state_interface name="position"/>
-    </joint>
-    <joint name="link_7_8_joint">
-        <command_interface name="effort">
-            <param name="min">0</param>
-            <param name="max">200</param>
-        </command_interface>
-        <state_interface name="position"/>
-    </joint>
-    <joint name="link_8_9_joint">
-        <command_interface name="effort">
-            <param name="min">0</param>
-            <param name="max">200</param>
-        </command_interface>
-        <state_interface name="position"/>
-    </joint>
-    <joint name="link_9_10_joint">
-        <command_interface name="effort">
-            <param name="min">0</param>
-            <param name="max">200</param>
-        </command_interface>
-        <state_interface name="position"/>
-    </joint>
-  </ros2_control>
+        <joint name="link_1_2_joint">
+            <command_interface name="effort">
+                <param name="min">0</param>
+                <param name="max">200</param>
+            </command_interface>
+            <state_interface name="position"/>
+        </joint>
+        <joint name="link_2_3_joint">
+            <command_interface name="effort">
+                <param name="min">0</param>
+                <param name="max">200</param>
+            </command_interface>
+            <state_interface name="position"/>
+        </joint>
+        <joint name="link_3_4_joint">
+            <command_interface name="effort">
+                <param name="min">0</param>
+                <param name="max">200</param>
+            </command_interface>
+            <state_interface name="position"/>
+        </joint>
+        <joint name="link_4_5_joint">
+            <command_interface name="effort">
+                <param name="min">0</param>
+                <param name="max">200</param>
+            </command_interface>
+            <state_interface name="position"/>
+        </joint>
+        <joint name="link_5_6_joint">
+            <command_interface name="effort">
+                <param name="min">0</param>
+                <param name="max">200</param>
+            </command_interface>
+            <state_interface name="position"/>
+        </joint>
+        <joint name="link_6_7_joint">
+            <command_interface name="effort">
+                <param name="min">0</param>
+                <param name="max">200</param>
+            </command_interface>
+            <state_interface name="position"/>
+        </joint>
+        <joint name="link_7_8_joint">
+            <command_interface name="effort">
+                <param name="min">0</param>
+                <param name="max">200</param>
+            </command_interface>
+            <state_interface name="position"/>
+        </joint>
+        <joint name="link_8_9_joint">
+            <command_interface name="effort">
+                <param name="min">0</param>
+                <param name="max">200</param>
+            </command_interface>
+            <state_interface name="position"/>
+        </joint>
+        <joint name="link_9_10_joint">
+            <command_interface name="effort">
+                <param name="min">0</param>
+                <param name="max">200</param>
+            </command_interface>
+            <state_interface name="position"/>
+        </joint>
+    </ros2_control>
     <gazebo>
-            <plugin name="gazebo_ros_planar_move" filename="libgazebo_ros_planar_move.so">
-                <update_rate>100</update_rate>
-                <publish_rate>10</publish_rate>
-                <!-- output -->
-                <publish_odom>true</publish_odom>
-                <publish_odom_tf>true</publish_odom_tf>
-                <odometry_frame>odom</odometry_frame>
-                <robot_base_frame>base_link</robot_base_frame>
-              </plugin>
+        <plugin name="gazebo_ros_planar_move" filename="libgazebo_ros_planar_move.so">
+            <update_rate>100</update_rate>
+            <publish_rate>10</publish_rate>
+            <!-- output -->
+            <publish_odom>true</publish_odom>
+            <publish_odom_tf>true</publish_odom_tf>
+            <odometry_frame>odom</odometry_frame>
+            <robot_base_frame>base_link</robot_base_frame>
+        </plugin>
         <plugin name="gazebo_ros2_control" filename="libgazebo_ros2_control.so">
-        <parameters>$(find snake_bot)/config/controllers.yaml</parameters>
+            <parameters>$(find snake_bot)/config/controllers.yaml</parameters>
         </plugin>
         <plugin name="ft_sensor" filename="libgazebo_ros_ft_sensor.so">

Commit message: obstacles, robot and gazebo view alligned

File: src/snake_bot/urdf/ros2_control.xacro (robot description, xacro)
@@ -11,23 +11,23 @@
     </gazebo>
     <gazebo reference="link_4">
-        <material>Gazebo/Blue</material>
+        <material>Gazebo/White</material>
     </gazebo>
     <gazebo reference="link_5">
-        <material>Gazebo/Green</material>
+        <material>Gazebo/Yellow</material>
     </gazebo>
     <gazebo reference="link_6">
-        <material>Gazebo/Blue</material>
+        <material>Gazebo/Purple</material>
     </gazebo>
     <gazebo reference="link_7">
-        <material>Gazebo/Orange</material>
+        <material>Gazebo/Black</material>
     </gazebo>
     <gazebo reference="link_8">
-        <material>Gazebo/Green</material>
+        <material>Gazebo/Indigo</material>
     </gazebo>
     <gazebo reference="link_9">
-        <material>Gazebo/Blue</material>
+        <material>Gazebo/RedBright</material>
     </gazebo>
     <gazebo reference="link_10">
-        <material>Gazebo/Orange</material>
+        <material>Gazebo/Turquoise</material>
     </gazebo>
     <ros2_control name="GazeboSystem" type="system">

File: src/snake_bot/urdf/snakebot.xacro (robot description, xacro)
@@ -12,10 +12,10 @@
       <parent link="base_link"/>
       <child link="link_1"/>
-      <origin xyz="0.0 0 0.0" rpy="0 0 0"/>
-     </joint>
+      <origin xyz="0.0 0 0.0" rpy="0 0 0.523599"/>
+    </joint>
     <!--LINK_1 -->
     <link name="link_1">
         <visual>
-            <origin xyz="0.0 0.07 0.03" rpy="0.0 0.0 0.0"/>
+            <origin xyz="0.0 0.07 0.03" rpy="0.0 0.0 0"/>
             <geometry>
                 <box size="0.06 0.14 0.06"/>
@@ -24,11 +24,11 @@
         </visual>
         <collision>
-            <origin xyz="0.0 0.07 0.03" rpy="0.0 0.0 0.0"/>
-            <geometry>
-                <box size="0.06 0.14 0.06"/>
-            </geometry>
-        </collision>
-        <xacro:inertial_box mass="1" x="0.06" y="0.14" z="0.06">
-            <origin xyz="0.0 0.07 0.03" rpy="0.0 0.0 0.0"/>
+            <origin xyz="0.0 0.07 0.03" rpy="0.0 0.0 0"/>
+            <geometry>
+                <box size="0.06 0.14 0.06"/>
+            </geometry>
+        </collision>
+        <xacro:inertial_box mass="1" x="0.06" y="0.14" z="0.06">
+            <origin xyz="0.0 0.07 0.03" rpy="0.0 0.0 0"/>
         </xacro:inertial_box>
     </link>
@@ -38,5 +38,5 @@
         <child link="link_2"/>
         <limit lower="-0.785398163397" upper="0.785398163397" velocity="50.0" effort="1000.0"/>
-        <origin xyz="0.0 0.175 0.0" rpy="0 0 0"/>
+        <origin xyz="0.0 0.175 0.0" rpy="0 0 -0.174533"/>
         <axis xyz="0 0 1"/>
         <joint_properties damping="6.0" friction="6.0"/>
@@ -66,5 +66,5 @@
         <child link="link_3"/>
         <limit lower="-0.785398163397" upper="0.785398163397" velocity="50.0" effort="1000.0"/>
-        <origin xyz="0.0 0.175 0.0" rpy="0 0 -1.309"/>
+        <origin xyz="0.0 0.175 0.0" rpy="0 0 -0.174533"/>
         <axis xyz="0 0 1"/>
         <joint_properties damping="6.0" friction="6.0"/>
@@ -94,5 +94,5 @@
         <child link="link_4"/>
         <limit lower="-0.785398163397" upper="0.785398163397" velocity="50.0" effort="1000.0"/>
-        <origin xyz="0.0 0.175 0.0" rpy="0 0 0"/>
+        <origin xyz="0.0 0.175 0.0" rpy="0 0 -0.174533"/>
         <axis xyz="0 0 1"/>
         <joint_properties damping="6.0" friction="6.0"/>
@@ -121,5 +121,5 @@
         <child link="link_5"/>
         <limit lower="-0.785398163397" upper="0.785398163397" velocity="50.0" effort="1000.0"/>
-        <origin xyz="0.0 0.175 0.0" rpy="0 0 0"/>
+        <origin xyz="0.0 0.175 0.0" rpy="0 0 -0.174533"/>
         <axis xyz="0 0 1"/>
         <joint_properties damping="6.0" friction="6.0"/>
@@ -148,5 +148,5 @@
         <child link="link_6"/>
         <limit lower="-0.785398163397" upper="0.785398163397" velocity="50.0" effort="1000.0"/>
-        <origin xyz="0.0 0.175 0.0" rpy="0 0 -1.22173"/>
+        <origin xyz="0.0 0.175 0.0" rpy="0 0 -0.174533"/>
         <axis xyz="0 0 1"/>
         <joint_properties damping="6.0" friction="6.0"/>
@@ -204,5 +204,5 @@
         <child link="link_8"/>
         <limit lower="-0.785398163397" upper="0.785398163397" velocity="50.0" effort="1000.0"/>
-        <origin xyz="0.0 0.175 0.0" rpy="0 0 -0.174533"/>
+        <origin xyz="0.0 0.175 0.0" rpy="0 0 0.174533"/>
         <axis xyz="0 0 1"/>
         <joint_properties damping="6.0" friction="6.0"/>
@@ -232,5 +232,5 @@
         <child link="link_9"/>
         <limit lower="-0.785398163397" upper="0.785398163397" velocity="50.0" effort="1000.0"/>
-        <origin xyz="0.0 0.175 0.0" rpy="0 0 -0.174533"/>
+        <origin xyz="0.0 0.175 0.0" rpy="0 0 0.174533"/>
         <axis xyz="0 0 1"/>
         <joint_properties damping="6.0" friction="6.0"/>
@@ -260,5 +260,5 @@
         <child link="link_10"/>
         <limit lower="-0.785398163397" upper="0.785398163397" velocity="50.0" effort="1000.0"/>
-        <origin xyz="0.0 0.175 0.0" rpy="0 0 -1.309"/>
+        <origin xyz="0.0 0.175 0.0" rpy="0 0 0.174533"/>
         <axis xyz="0 0 1"/>
         <joint_properties damping="6.0" friction="6.0"/>
