Commit message: sensors worknig and configured for all elementst

File: src/snake_bot/urdf/ros2_control.xacro (robot description, xacro)
@@ -3,31 +3,171 @@
     <gazebo reference="link_1">
         <material>Gazebo/Green</material>
+        <sensor name="link1_contact_sensor" type="contact">
+            <always_on>true</always_on>
+            <contact>
+                <collision>link_1_collision_collision</collision>
+            </contact>
+            <update_rate>1</update_rate>
+            <plugin name="link1_bumper_plugin" filename="libgazebo_ros_bumper.so">
+                <frame_name>world</frame_name>
+                <bumperTopicName>link1_bumper</bumperTopicName>
+                <ros>
+                    <remapping>bumper_states:=link1_bumper_states</remapping>
+                </ros>
+            </plugin>
+        </sensor>
     </gazebo>
     <gazebo reference="link_2">
         <material>Gazebo/Blue</material>
+        <sensor name="link2_contact_sensor" type="contact">
+            <always_on>true</always_on>
+            <contact>
+                <collision>link_2_collision_collision</collision>
+            </contact>
+            <update_rate>1</update_rate>
+            <plugin name="link2_bumper_plugin" filename="libgazebo_ros_bumper.so">
+                <frame_name>world</frame_name>
+                <bumperTopicName>link2_bumper</bumperTopicName>
+                <ros>
+                    <remapping>bumper_states:=link2_bumper_states</remapping>
+                </ros>
+            </plugin>
+        </sensor>
     </gazebo>
     <gazebo reference="link_3">
         <material>Gazebo/Orange</material>
+        <sensor name="link3_contact_sensor" type="contact">
+            <always_on>true</always_on>
+            <contact>
+                <collision>link_3_collision_collision</collision>
+            </contact>
+            <update_rate>1</update_rate>
+            <plugin name="link3_bumper_plugin" filename="libgazebo_ros_bumper.so">
+                <frame_name>world</frame_name>
+                <bumperTopicName>link3_bumper</bumperTopicName>
+                <ros>
+                    <remapping>bumper_states:=link3_bumper_states</remapping>
+                </ros>
+            </plugin>
+        </sensor>
     </gazebo>
     <gazebo reference="link_4">
         <material>Gazebo/White</material>
+        <sensor name="link4_contact_sensor" type="contact">
+            <always_on>true</always_on>
+            <contact>
+                <collision>link_4_collision_collision</collision>
+            </contact>
+            <update_rate>1</update_rate>
+            <plugin name="link4_bumper_plugin" filename="libgazebo_ros_bumper.so">
+                <frame_name>world</frame_name>
+                <bumperTopicName>link4_bumper</bumperTopicName>
+                <ros>
+                    <remapping>bumper_states:=link4_bumper_states</remapping>
+                </ros>
+            </plugin>
+        </sensor>
     </gazebo>
     <gazebo reference="link_5">
         <material>Gazebo/Yellow</material>
+        <sensor name="link5_contact_sensor" type="contact">
+            <always_on>true</always_on>
+            <contact>
+                <collision>link_5_collision_collision</collision>
+            </contact>
+            <update_rate>1</update_rate>
+            <plugin name="link5_bumper_plugin" filename="libgazebo_ros_bumper.so">
+                <frame_name>world</frame_name>
+                <bumperTopicName>link5_bumper</bumperTopicName>
+                <ros>
+                    <remapping>bumper_states:=link5_bumper_states</remapping>
+                </ros>
+            </plugin>
+        </sensor>
     </gazebo>
     <gazebo reference="link_6">
         <material>Gazebo/Purple</material>
+        <sensor name="link6_contact_sensor" type="contact">
+            <always_on>true</always_on>
+            <contact>
+                <collision>link_6_collision_collision</collision>
+            </contact>
+            <update_rate>1</update_rate>
+            <plugin name="link6_bumper_plugin" filename="libgazebo_ros_bumper.so">
+                <frame_name>world</frame_name>
+                <bumperTopicName>link6_bumper</bumperTopicName>
+                <ros>
+                    <remapping>bumper_states:=link6_bumper_states</remapping>
+                </ros>
+            </plugin>
+        </sensor>
     </gazebo>
     <gazebo reference="link_7">
         <material>Gazebo/Black</material>
+        <sensor name="link7_contact_sensor" type="contact">
+            <always_on>true</always_on>
+            <contact>
+                <collision>link_7_collision_collision</collision>
+            </contact>
+            <update_rate>1</update_rate>
+            <plugin name="link7_bumper_plugin" filename="libgazebo_ros_bumper.so">
+                <frame_name>world</frame_name>
+                <bumperTopicName>link7_bumper</bumperTopicName>
+                <ros>
+                    <remapping>bumper_states:=link7_bumper_states</remapping>
+                </ros>
+            </plugin>
+        </sensor>
     </gazebo>
     <gazebo reference="link_8">
         <material>Gazebo/Indigo</material>
+        <sensor name="link8_contact_sensor" type="contact">
+            <always_on>true</always_on>
+            <contact>
+                <collision>link_8_collision_collision</collision>
+            </contact>
+            <update_rate>1</update_rate>
+            <plugin name="link8_bumper_plugin" filename="libgazebo_ros_bumper.so">
+                <frame_name>world</frame_name>
+                <bumperTopicName>link8_bumper</bumperTopicName>
+                <ros>
+                    <remapping>bumper_states:=link8_bumper_states</remapping>
+                </ros>
+            </plugin>
+        </sensor>
     </gazebo>
     <gazebo reference="link_9">
         <material>Gazebo/RedBright</material>
+        <sensor name="link9_contact_sensor" type="contact">
+            <always_on>true</always_on>
+            <contact>
+                <collision>link_9_collision_collision</collision>
+            </contact>
+            <update_rate>1</update_rate>
+            <plugin name="link9_bumper_plugin" filename="libgazebo_ros_bumper.so">
+                <frame_name>world</frame_name>
+                <bumperTopicName>link9_bumper</bumperTopicName>
+                <ros>
+                    <remapping>bumper_states:=link9_bumper_states</remapping>
+                </ros>
+            </plugin>
+        </sensor>
     </gazebo>
     <gazebo reference="link_10">
         <material>Gazebo/Turquoise</material>
+        <sensor name="link10_contact_sensor" type="contact">
+            <always_on>true</always_on>
+            <contact>
+                <collision>link_10_collision_collision</collision>
+            </contact>
+            <update_rate>1</update_rate>
+            <plugin name="link10_bumper_plugin" filename="libgazebo_ros_bumper.so">
+                <frame_name>world</frame_name>
+                <bumperTopicName>link10_bumper</bumperTopicName>
+                <ros>
+                    <remapping>bumper_states:=link10_bumper_states</remapping>
+                </ros>
+            </plugin>
+        </sensor>
     </gazebo>
     <ros2_control name="GazeboSystem" type="system">
@@ -35,5 +175,4 @@
             <plugin>gazebo_ros2_control/GazeboSystem</plugin>
     	</hardware>
-<!--  ****************************************************** * * * BELOW IS Commented * *************************************************************************************** * * * * * -->
         <joint name="link_1_2_joint">
             <command_interface name="effort">
@@ -113,5 +252,5 @@
             <parameters>$(find snake_bot)/config/controllers.yaml</parameters>
         </plugin>
-        <plugin name="ft_sensor" filename="libgazebo_ros_ft_sensor.so">
+        <plugin name="ft_sensor_joint_1" filename="libgazebo_ros_ft_sensor.so">
             <updateRate>100.0</updateRate>
             <remapping>wrench:=joint_1</remapping>
@@ -120,4 +259,60 @@
             <update_rate>1</update_rate>
         </plugin>
+        <plugin name="ft_sensor_joint_2" filename="libgazebo_ros_ft_sensor.so">
+            <updateRate>100.0</updateRate>
+            <remapping>wrench:=joint_2</remapping>
+            <joint_name>link_2_3_joint</joint_name>
+            <gaussian_noise>0.01</gaussian_noise>
+            <update_rate>1</update_rate>
+        </plugin>
+        <plugin name="ft_sensor_joint_3" filename="libgazebo_ros_ft_sensor.so">
+            <updateRate>100.0</updateRate>
+            <remapping>wrench:=joint_3</remapping>
+            <joint_name>link_3_4_joint</joint_name>
+            <gaussian_noise>0.01</gaussian_noise>
+            <update_rate>1</update_rate>
+        </plugin>
+        <plugin name="ft_sensor_joint_4" filename="libgazebo_ros_ft_sensor.so">
+            <updateRate>100.0</updateRate>
+            <remapping>wrench:=joint_4</remapping>
+            <joint_name>link_4_5_joint</joint_name>
+            <gaussian_noise>0.01</gaussian_noise>
+            <update_rate>1</update_rate>
+        </plugin>
+        <plugin name="ft_sensor_joint_5" filename="libgazebo_ros_ft_sensor.so">
+            <updateRate>100.0</updateRate>
+            <remapping>wrench:=joint_5</remapping>
+            <joint_name>link_5_6_joint</joint_name>
+            <gaussian_noise>0.01</gaussian_noise>
+            <update_rate>1</update_rate>
+        </plugin>
+        <plugin name="ft_sensor_joint_6" filename="libgazebo_ros_ft_sensor.so">
+            <updateRate>100.0</updateRate>
+            <remapping>wrench:=joint_6</remapping>
+            <joint_name>link_6_7_joint</joint_name>
+            <gaussian_noise>0.01</gaussian_noise>
+            <update_rate>1</update_rate>
+        </plugin>
+        <plugin name="ft_sensor_joint_7" filename="libgazebo_ros_ft_sensor.so">
+            <updateRate>100.0</updateRate>
+            <remapping>wrench:=joint_7</remapping>
+            <joint_name>link_7_8_joint</joint_name>
+            <gaussian_noise>0.01</gaussian_noise>
+            <update_rate>1</update_rate>
+        </plugin>
+        <plugin name="ft_sensor_joint_8" filename="libgazebo_ros_ft_sensor.so">
+            <updateRate>100.0</updateRate>
+            <remapping>wrench:=joint_8</remapping>
+            <joint_name>link_8_9_joint</joint_name>
+            <gaussian_noise>0.01</gaussian_noise>
+            <update_rate>1</update_rate>
+        </plugin>
+        <plugin name="ft_sensor_joint_9" filename="libgazebo_ros_ft_sensor.so">
+            <updateRate>100.0</updateRate>
+            <remapping>wrench:=joint_9</remapping>
+            <joint_name>link_9_10_joint</joint_name>
+            <gaussian_noise>0.01</gaussian_noise>
+            <update_rate>1</update_rate>
+        </plugin>
     </gazebo>
 </robot>

Commit message: trying to sync subscribers before calculation

File: src/snake_bot/urdf/ros2_control.xacro (robot description, xacro)
@@ -6,5 +6,5 @@
             <always_on>true</always_on>
             <contact>
-                <collision>link_1_collision_collision</collision>
+                <collision>base_link_fixed_joint_lump__link_1_collision_collision</collision>
             </contact>
             <update_rate>1</update_rate>
@@ -15,4 +15,5 @@
                     <remapping>bumper_states:=link1_bumper_states</remapping>
                 </ros>
+                <updateRate>1.0</updateRate>
             </plugin>
         </sensor>
@@ -32,4 +33,5 @@
                     <remapping>bumper_states:=link2_bumper_states</remapping>
                 </ros>
+                <updateRate>1.0</updateRate>
             </plugin>
         </sensor>
@@ -49,4 +51,5 @@
                     <remapping>bumper_states:=link3_bumper_states</remapping>
                 </ros>
+                <updateRate>1.0</updateRate>
             </plugin>
         </sensor>
@@ -66,4 +69,5 @@
                     <remapping>bumper_states:=link4_bumper_states</remapping>
                 </ros>
+                <updateRate>1.0</updateRate>
             </plugin>
         </sensor>
@@ -83,4 +87,5 @@
                     <remapping>bumper_states:=link5_bumper_states</remapping>
                 </ros>
+                <updateRate>1.0</updateRate>
             </plugin>
         </sensor>
@@ -100,4 +105,5 @@
                     <remapping>bumper_states:=link6_bumper_states</remapping>
                 </ros>
+                <updateRate>1.0</updateRate>
             </plugin>
         </sensor>
@@ -117,4 +123,5 @@
                     <remapping>bumper_states:=link7_bumper_states</remapping>
                 </ros>
+                <updateRate>1.0</updateRate>
             </plugin>
         </sensor>
@@ -134,4 +141,5 @@
                     <remapping>bumper_states:=link8_bumper_states</remapping>
                 </ros>
+                <updateRate>1.0</updateRate>
             </plugin>
         </sensor>
@@ -151,4 +159,5 @@
                     <remapping>bumper_states:=link9_bumper_states</remapping>
                 </ros>
+                <updateRate>1.0</updateRate>
             </plugin>
         </sensor>
@@ -168,4 +177,5 @@
                     <remapping>bumper_states:=link10_bumper_states</remapping>
                 </ros>
+                <updateRate>1.0</updateRate>
             </plugin>
         </sensor>

Commit message: new controller with sign wave

File: src/snake_bot/urdf/ros2_control.xacro (robot description, xacro)
@@ -270,4 +270,9 @@
         <plugin name="gazebo_ros2_control" filename="libgazebo_ros2_control.so">
             <parameters>$(find snake_bot)/config/controllers.yaml</parameters>
+            <robot_sim_type>gazebo_ros2_control/GazeboSystem</robot_sim_type>
+            <type>controller_manager/ControllerManager</type>
+            <!-- Add joint state publishing -->
+            <publish_joint_states>true</publish_joint_states>
+            <joint_state_topic>joint_states</joint_state_topic>
         </plugin>
         <plugin name="ft_sensor_joint_1" filename="libgazebo_ros_ft_sensor.so">

File: src/snake_bot/urdf/snakebot.xacro (robot description, xacro)
@@ -12,5 +12,5 @@
       <parent link="base_link"/>
       <child link="link_1"/>
-      <origin xyz="0.0 0 0.0" rpy="0 0 0.436332"/>
+      <origin xyz="0.0 0 0.0" rpy="0 0 0"/>
     </joint>
     <!--LINK_1 -->
@@ -38,5 +38,5 @@
         <child link="link_2"/>
         <limit lower="-0.785398163397" upper="0.785398163397" velocity="50.0" effort="1000.0"/>
-        <origin xyz="0.0 0.175 0.0" rpy="0 0 -0.174533"/>
+        <origin xyz="0.0 0.175 0.0" rpy="0 0 0"/>
         <axis xyz="0 0 1"/>
         <joint_properties damping="6.0" friction="6.0"/>
@@ -66,5 +66,5 @@
         <child link="link_3"/>
         <limit lower="-0.785398163397" upper="0.785398163397" velocity="50.0" effort="1000.0"/>
-        <origin xyz="0.0 0.175 0.0" rpy="0 0 -0.174533"/>
+        <origin xyz="0.0 0.175 0.0" rpy="0 0 0"/>
         <axis xyz="0 0 1"/>
         <joint_properties damping="6.0" friction="6.0"/>
@@ -94,5 +94,5 @@
         <child link="link_4"/>
         <limit lower="-0.785398163397" upper="0.785398163397" velocity="50.0" effort="1000.0"/>
-        <origin xyz="0.0 0.175 0.0" rpy="0 0 -0.174533"/>
+        <origin xyz="0.0 0.175 0.0" rpy="0 0 0"/>
         <axis xyz="0 0 1"/>
         <joint_properties damping="6.0" friction="6.0"/>
@@ -121,5 +121,5 @@
         <child link="link_5"/>
         <limit lower="-0.785398163397" upper="0.785398163397" velocity="50.0" effort="1000.0"/>
-        <origin xyz="0.0 0.175 0.0" rpy="0 0 -0.174533"/>
+        <origin xyz="0.0 0.175 0.0" rpy="0 0 0"/>
         <axis xyz="0 0 1"/>
         <joint_properties damping="6.0" friction="6.0"/>
@@ -148,5 +148,5 @@
         <child link="link_6"/>
         <limit lower="-0.785398163397" upper="0.785398163397" velocity="50.0" effort="1000.0"/>
-        <origin xyz="0.0 0.175 0.0" rpy="0 0 -0.174533"/>
+        <origin xyz="0.0 0.175 0.0" rpy="0 0 0"/>
         <axis xyz="0 0 1"/>
         <joint_properties damping="6.0" friction="6.0"/>
@@ -204,5 +204,5 @@
         <child link="link_8"/>
         <limit lower="-0.785398163397" upper="0.785398163397" velocity="50.0" effort="1000.0"/>
-        <origin xyz="0.0 0.175 0.0" rpy="0 0 0.174533"/>
+        <origin xyz="0.0 0.175 0.0" rpy="0 0 0"/>
         <axis xyz="0 0 1"/>
         <joint_properties damping="6.0" friction="6.0"/>
@@ -232,5 +232,5 @@
         <child link="link_9"/>
         <limit lower="-0.785398163397" upper="0.785398163397" velocity="50.0" effort="1000.0"/>
-        <origin xyz="0.0 0.175 0.0" rpy="0 0 0.174533"/>
+        <origin xyz="0.0 0.175 0.0" rpy="0 0 0"/>
         <axis xyz="0 0 1"/>
         <joint_properties damping="6.0" friction="6.0"/>
@@ -260,5 +260,5 @@
         <child link="link_10"/>
         <limit lower="-0.785398163397" upper="0.785398163397" velocity="50.0" effort="1000.0"/>
-        <origin xyz="0.0 0.175 0.0" rpy="0 0 0.174533"/>
+        <origin xyz="0.0 0.175 0.0" rpy="0 0 0"/>
         <axis xyz="0 0 1"/>
         <joint_properties damping="6.0" friction="6.0"/>
